Commit message: change sth

File: mobile/urdf/mobile.urdf (robot description, URDF)
Before this commit: robot mobile, 14 links, 13 joints
Joints:
- joint left_wheel_jn: type continuous -> fixed
- joint phaisau_duoi_jn: type continuous -> fixed
- joint phaisau_tren_jn: type continuous -> fixed
- joint right_wheel_jn: type continuous -> fixed
- joint traisau_duoi_jn: type continuous -> fixed
- joint traisau_tren_jn: type continuous -> fixed
- joint truocphai_duoi_jn: type continuous -> fixed
- joint truocphai_tren_jn: type continuous -> fixed
- joint truoctrai_duoi_jn: type continuous -> fixed
- joint truoctrai_tren_jn: type continuous -> fixed

Commit message: Clean ROS2 build files and update mobile robot project

File: mobile/urdf/mobile.urdf (robot description, URDF)
Before this commit: robot mobile, 14 links, 13 joints
Links:
- added link camera_high_color_frame
- added link camera_high_color_optical_frame
- added link camera_high_depth_frame
- added link camera_high_depth_optical_frame
- added link camera_high_link; visual box size=0.03 0.03 0.03
- added link camera_low_depth_frame
- added link camera_low_depth_optical_frame
- added link camera_low_ir_frame
- added link camera_low_ir_optical_frame
- added link camera_low_link; visual box size=0.09 0.025 0.025
Joints:
- added joint camera_high_color_frame_joint: type fixed, parent camera_high_link, child camera_high_color_frame, origin xyz=0 0 0 rpy=0 0 0
- added joint camera_high_color_optical_frame_joint: type fixed, parent camera_high_color_frame, child camera_high_color_optical_frame, origin xyz=0 0 0 rpy=-1.570796 0 -1.570796
- added joint camera_high_depth_frame_joint: type fixed, parent camera_high_link, child camera_high_depth_frame, origin xyz=0 0 0 rpy=0 0 0
- added joint camera_high_depth_optical_frame_joint: type fixed, parent camera_high_depth_frame, child camera_high_depth_optical_frame, origin xyz=0 0 0 rpy=-1.570796 0 -1.570796
- added joint camera_high_joint: type fixed, parent base_link, child camera_high_link, origin xyz=0.325 0 0.33 rpy=0 0 0
- added joint camera_low_depth_frame_joint: type fixed, parent camera_low_link, child camera_low_depth_frame, origin xyz=0 0 0 rpy=0 0 0
- added joint camera_low_depth_optical_frame_joint: type fixed, parent camera_low_depth_frame, child camera_low_depth_optical_frame, origin xyz=0 0 0 rpy=-1.570796 0 -1.570796
- added joint camera_low_ir_frame_joint: type fixed, parent camera_low_depth_frame, child camera_low_ir_frame, origin xyz=0 0 0 rpy=0 0 0
- added joint camera_low_ir_optical_frame_joint: type fixed, parent camera_low_ir_frame, child camera_low_ir_optical_frame, origin xyz=0 0 0 rpy=-1.570796 0 -1.570796
- added joint camera_low_joint: type fixed, parent base_link, child camera_low_link, origin xyz=0.375 0.0 1.1 rpy=0.0 0.785 0.0
